File: hardware/main/controller-support.kicad_sch (KiCad schematic)
At the start: 14 parts, among them SW1 ESP RESET, SW2 ESP BOOT

Commit message: PCB housing
Parts:
- removed R4: 10k, Resistor_SMD:R_0402_1005Metric, symbol Device:R
- removed SW1: ESP RESET, Button_Switch_SMD:SW_SPST_TL3305A, symbol Switch:SW_Push
- removed SW2: ESP BOOT, Button_Switch_SMD:SW_SPST_TL3305A, symbol Switch:SW_Push
- added J3: ESP RECOVERY, HapticBracelet:ESP_Recovery_3Pads_P1.5mm, symbol Connector_Generic:Conn_01x03
Connections:
- net BOOT_IO9: now also J3.3 (Pin_3)
- net GND: now also J3.2 (Pin_2)
- net MCU_EN: now also J3.1 (Pin_1)
Other:
- note added: "UNDERSIDE RECOVERY PADS: 1 EN / 2 GND / 3 BOOT Hold BOOT low; pulse EN low; release EN, then BOOT."
- moved on the sheet: C1, R3
