File: hardware/main/main.kicad_sch (KiCad schematic)
At the start: 9 parts, among them U1 ESP32-C6-MINI-1, U26 TPS22918DBV

Commit message: PCB housing
Parts:
- added R4: 10k, Resistor_SMD:R_0402_1005Metric, symbol Device:R
Connections:
- net +3V3: now also R4.1
- net BOOT_IO8: now also R4.2
Other:
- sheet Local haptic pod and harness renamed Stacked universal pod interface
- sheet Stacked universal pod interface: file local-pod.kicad_sch -> pod-interface.kicad_sch
- note added: "250 kbaud ring: ESP TX -> J101 -> universal pod 0 -> ... -> pod 7 -> RETURN -> ESP RX. 8 identical pod PCBAs + 1 controller daughterboard; protected batteries/NTCs on pods 1-7 only."
- note added: "HAPTIC BRACELET / CONTROLLER DAUGHTERBOARD"
- note removed: "250 kbaud logical ring: ESP TX -> pod 0 -> ... -> pod 7 -> RETURN -> ESP RX. Physical five-wire chain; RETURN runs back through the same links. No electrical connection across clasp."
- note removed: "HAPTIC BRACELET / MAIN PCBA"
- title: Controller and switched pod power -> Haptic bracelet - stacked controller
Changed lines of the file:
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@@
 	(paper "A3")
 	(title_block
-		(title "Controller and switched pod power")
-		(date "2026-09-12")
+		(title "Haptic bracelet - stacked controller")
+		(date "2026-09-14")
 		(rev "0.5")
 		(comment 1 "One wrist / ring pod schematic draft")
@@
 		)
 	)
-	(text "250 kbaud logical ring: ESP TX -> pod 0 -> ... -> pod 7 -> RETURN -> ESP RX.\nPhysical five-wire chain; RETURN runs back through the same links. No electrical connection across clasp."
+	(text "250 kbaud ring: ESP TX -> J101 -> universal pod 0 -> ... -> pod 7 -> RETURN -> ESP RX.\n8 identical pod PCBAs + 1 controller daughterboard; protected batteries/NTCs on pods 1-7 only."
 		(exclude_from_sim no)
 		(at 15.24 22.86 0)
@@
 		)
 	)
-	(text "HAPTIC BRACELET / MAIN PCBA"
+	(text "HAPTIC BRACELET / CONTROLLER DAUGHTERBOARD"
 		(exclude_from_sim no)
 		(at 15.24 12.7 0)
@@
 	)
 	(junction
+		(at 34.29 88.9)
+		(diameter 0)
+		(color 0 0 0 0)
+	)
+	(junction
 		(at 107.95 193.04)
 		(diameter 0)
@@
 	(wire
 		(pts
+			(xy 34.29 88.9) (xy 34.29 83.82)
+		)
+		(stroke
+			(width 0)
+			(type default)
+		)
+	)
+	(wire
+		(pts
 			(xy 123.19 196.85) (xy 123.19 193.04)
 		)
@@
 	(wire
 		(pts
-			(xy 58.42 88.9) (xy 53.34 88.9)
+			(xy 34.29 76.2) (xy 34.29 71.12)
 		)
 		(stroke
@@
 	(wire
 		(pts
+			(xy 34.29 88.9) (xy 58.42 88.9)
+		)
+		(stroke
+			(width 0)
+			(type default)
+		)
+	)
+	(wire
+		(pts
 			(xy 58.42 91.44) (xy 53.34 91.44)
 		)
@@
 		(pts
 			(xy 45.72 187.96) (xy 45.72 193.04)
+		)
+		(stroke
+			(width 0)
+			(type default)
+		)
+	)
+	(wire
+		(pts
+			(xy 33.02 88.9) (xy 34.29 88.9)
 		)
 		(stroke
@@
 		)
 	)
+	(global_label "BOOT_IO8"
+		(shape bidirectional)
+		(at 33.02 88.9 180)
+		(effects
+			(font
+				(size 1 1)
+			)
+			(justify right bottom)
+		)
+		(property "Intersheetrefs" "${INTERSHEET_REFS}"
+			(at 33.02 88.9 0)
+			(hide yes)
+			(show_name no)
+			(do_not_autoplace no)
+			(effects
+				(font
+					(size 1.27 1.27)
+				)
+				(justify left)
+			)
+		)
+	)
 	(global_label "LED_G_N"
 		(shape bidirectional)
@@
 		(property "Intersheetrefs" "${INTERSHEET_REFS}"
 			(at 93.98 91.44 0)
-			(hide yes)
-			(show_name no)
-			(do_not_autoplace no)
-			(effects
-				(font
-					(size 1.27 1.27)
-				)
-			)
-		)
-	)
-	(global_label "BOOT_IO8"
-		(shape bidirectional)
-		(at 53.34 88.9 180)
-		(effects
-			(font
-				(size 1 1)
-			)
-			(justify right bottom)
-		)
-		(property "Intersheetrefs" "${INTERSHEET_REFS}"
-			(at 53.34 88.9 0)
 			(hide yes)
 			(show_name no)
@@
 	)
 	(symbol
+		(lib_id "Device:R")
+		(at 34.29 80.01 0)
+		(unit 1)
+		(body_style 1)
+		(exclude_from_sim no)
+		(in_bom yes)
+		(on_board yes)
+		(in_pos_files yes)
+		(dnp no)
+		(property "Reference" "R4"
+			(at 37.29 78.74 0)
+			(show_name no)
+			(do_not_autoplace no)
+			(effects
+				(font
+					(size 1 1)
+				)
+				(justify left)
+			)
+		)
+		(property "Value" "10k"
+			(at 37.29 81.28 0)
+			(show_name no)
+			(do_not_autoplace no)
+			(effects
+				(font
+					(size 1 1)
+				)
+				(justify left)
+			)
+		)
+		(property "Footprint" "Resistor_SMD:R_0402_1005Metric"
+			(at -63.5 91.44 0)
+			(hide yes)
+			(show_name no)
+			(do_not_autoplace no)
+			(effects
+				(font
+					(size 1 1)
+				)
+			)
+		)
+		(property "Datasheet" ""
+			(at -63.5 91.44 0)
+			(hide yes)
+			(show_name no)
+			(do_not_autoplace no)
+			(effects
+				(font
+					(size 1 1)
+				)
+			)
+		)
+		(property "Description" ""
+			(at -67.31 90.17 0)
+			(show_name no)
+			(do_not_autoplace no)
+			(effects
+				(font
+					(size 1.27 1.27)
+				)
+			)
+		)
+		(pin "1"
+		)
+		(pin "2"
+		)
+		(instances
+			(project "main"
+				(path "/281e434a-bf9f-4327-92ec-86d5315beda6"
+					(reference "R4")
+					(unit 1)
+				)
+			)
+		)
+	)
+	(symbol
 		(lib_id "power:GND")
 		(at 114.3 104.14 0)
@@
 	)
 	(symbol
+		(lib_id "power:+3V3")
+		(at 34.29 71.12 0)
+		(unit 1)
+		(body_style 1)
+		(exclude_from_sim no)
+		(in_bom no)
+		(on_board yes)
+		(in_pos_files yes)
+		(dnp no)
+		(property "Reference" "#PWR030017"
+			(at 34.29 71.12 0)
+			(hide yes)
+			(show_name no)
+			(do_not_autoplace no)
+			(effects
+				(font
+					(size 1 1)
+				)
+			)
+		)
+		(property "Value" "+3V3"
+			(at 34.29 67.31 0)
+			(show_name no)
+			(do_not_autoplace no)
+			(effects
+				(font
+					(size 1 1)
+				)
+			)
+		)
+		(property "Footprint" ""
+			(at 34.29 71.12 0)
+			(show_name no)
+			(do_not_autoplace no)
+			(effects
+				(font
+					(size 1.27 1.27)
+				)
+			)
+		)
+		(property "Datasheet" ""
+			(at 34.29 71.12 0)
+			(show_name no)
+			(do_not_autoplace no)
+			(effects
+				(font
+					(size 1.27 1.27)
+				)
+			)
+		)
+		(property "Description" ""
+			(at 34.29 71.12 0)
+			(show_name no)
+			(do_not_autoplace no)
+			(effects
+				(font
+					(size 1.27 1.27)
+				)
+			)
+		)
+		(pin "1"
+		)
+		(instances
+			(project "main"
+				(path "/281e434a-bf9f-4327-92ec-86d5315beda6"
+					(reference "#PWR030017")
+					(unit 1)
+				)
+			)
+		)
+	)
+	(symbol
 		(lib_id "power:GND")
 		(at 52.07 226.06 0)
@@
 			(color 0 0 0 0)
 		)
-		(property "Sheetname" "Local haptic pod and harness"
+		(property "Sheetname" "Stacked universal pod interface"
 			(at 294.64 48.26 0)
 			(show_name no)
@@
 			)
 		)
-		(property "Sheetfile" "local-pod.kicad_sch"
+		(property "Sheetfile" "pod-interface.kicad_sch"
 			(at 294.64 78.74 0)
 			(show_name no)
