File: hardware/main/power.kicad_sch (KiCad schematic)
At the start: 17 parts, among them Q1 2N7002, SW3 WAKE / SHIP, U11 BQ25186DLH, U12 TPS63802DLA

Commit message: PCB housing
Parts:
- Q1: footprint Package_TO_SOT_SMD:SOT-23 -> Package_TO_SOT_SMD:SOT-323_SC-70
- SW3: footprint Button_Switch_SMD:Panasonic_EVQPUJ_EVQPUA -> HapticBracelet:SW_SPST_Panasonic_EVPAW_3x2mm_H0.6mm; BOM Comments Momentary TS/MR button per charger application; long-press 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 -> Outward-facing top-push SW3; EVPAWBD4A, 1.6 N, 0.6 mm heigh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; MPN EVQPUJ02K -> EVPAWBD4A
Other:
- note added: "C34: IN bypass C35: SYS reservoir C36: BAT bypass SW3: wake/ship button. R62: fixed TS/MR termination. VBAT arrives through J101 from seven protected cells on pods 1-7. No cell or NTC in pod 0. Require fresh temperatures from pods 1-7 before charge."
- note removed: "C34: IN bypass C35: SYS reservoir C36: BAT bypass SW3: wake/ship button. R62: fixed TS/MR termination. Cell and NTC use J200/J103 on the local pod sheet, as on satellites. Firmware checks every pod temperature before enabling charge."
