File: hardware/main/usb.kicad_sch (KiCad schematic)
At the start: 8 parts, among them J2 USB4105-GF-A, U14 TPD2EUSB30, U15 TPD2EUSB30

Commit message: PCB housing
Parts:
- removed U15: TPD2EUSB30, Package_TO_SOT_SMD:Texas_DRT-3, symbol Power_Protection:TPD2EUSB30
Other:
- moved on the sheet: R60, R61
