File: hardware/satellite/satellite.kicad_sch (KiCad schematic)
At the start: 24 parts, among them J1 CHAIN IN, J2 CHAIN OUT, J3 ICE / INITIAL FLASH, J4 PROTECTED CELL 90mAh, J5 NTC (optional), M1 VLV041235L, U1 M2003FC1AE, U2 DRV2625

Commit message: PCB housing
Parts:
- removed J3: ICE / INITIAL FLASH, HapticBracelet:WirePads_5_P1.27mm, symbol Connector_Generic:Conn_01x05
- added H1, H2, H3, H4: M1.6 STANDOFF, HapticBracelet:SMT_Standoff_M1p6_D3p3_ClosedBase_HeightTBD, symbol Mechanical:MountingHole
- added J6: Conn_ARM_SWD_TagConnect_TC2030-NL, Connector:Tag-Connect_TC2030-IDC-NL_2x03_P1.27mm_Vertical, symbol Connector:Conn_ARM_SWD_TagConnect_TC2030-NL
Connections:
- net +3V3_POD: now also J6.1 (VCC)
- net GND: now also J6.5 (GND)
- net LOCAL_nRESET: now also J6.3 (~{RESET})
- net UART_RX_LOCAL: now also J6.4 (SWCLK)
- net UART_TX_LOCAL: now also J6.2 (SWDIO)
- no-connect marks 13 -> 14
Other:
- note added: "ASSEMBLY: eight identical pod PCBAs per wrist. Pod 0 stacks beneath the controller; leave J4 battery and J5 NTC unwired. Pods 1-7 fit protected cells and NTCs. JP1 NORMAL on pods 0-6; END on pod 7."
- note added: "H1-H4: four corner M1.6 mounts. 20 x 46 mm PCB faces / TPU spacer. Standoff height and screw length TBD."
